File: eagle/master.sch (EAGLE design)
At the start: 15 parts

Commit message: Linear Regulators
Parts:
- added U1: TPS73633DBVR, TPS73633DBVR:TPS73633DBVR
Changed lines of the file:
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@@
 <part name="SUPPLY7" library="supply2" deviceset="DGND" device=""/>
 <part name="SUPPLY8" library="supply2" deviceset="DGND" device=""/>
+<part name="U1" library="TPS73633DBVR" deviceset="TPS73633DBVR" device=""/>
 </parts>
 <sheets>
@@
 </nets>
 </sheet>
+<sheet>
+<plain>
+</plain>
+<instances>
+<instance part="U1" gate="U1" x="58.42" y="88.9"/>
+</instances>
+<busses>
+</busses>
+<nets>
+</nets>
+</sheet>
