File: eagle/master2.sch (EAGLE design)
At the start: 16 parts, among them U1 TPS73633DBVR

Commit message: Microcontoller Schem
Parts:
- removed C1_V1, C1_V2, C1_V3, C1_V4, C1_V5, C1_V6: .1 uF, rcl:C-USC1206
- removed C2_V1, C2_V2, C2_V3, C2_V4, C2_V5, C2_V6: 4.7 uF, rcl:C-USC1206
- removed U1: TPS73633DBVR, TPS73633DBVR:TPS73633DBVR
- removed VCAP1, VCAP2: 2.2 uF, rcl:C-USC1206
- added C1: 4.7uF, rcl:C-USC1206
- added C10, C11, C12, C5, C8, C9: 100nF, rcl:C-USC1206
- added C2: 1uF, rcl:C-USC1206
- added C3, C4: 2.2uF, rcl:C-USC1206
- U$1: value LQFP100 -> STM32F767VG(2); device stmc7:LQFP100 -> MCU:STM32F767VG(2)
Connections:
- removed net AGND: C1_V6.2, C2_V6.2, U$1.VSSA
- removed net DGND: C1_V1.2, C1_V2.2, C1_V3.2, C1_V5.2, C2_V1.2, C2_V2.2, C2_V3.2, C2_V5.2, U$1.VSS@1, U$1.VSS@2, U$1.VSS@3, U$1.VSS@5, VCAP1.2, VCAP2.2
- removed net N$1: U$1.VCAP1, VCAP1.1
- removed net N$11: C1_V1.1, C2_V1.1, U$1.VDD@1
- removed net N$13: C1_V5.1, C2_V5.1, U$1.VDD@5
- removed net N$17: U$1.VBAT
- removed net N$2: U$1.VCAP2, VCAP2.1
- removed net N$5: C1_V2.1, C2_V2.1, U$1.VDD@2
- removed net N$7: C1_V4.1, C2_V4.1, U$1.VDD@4
- removed net N$8: C1_V4.2, C2_V4.2, U$1.VSS@4
- new net GND: C1.2, C10.2, C11.2, C12.2, C2.2, C3.2, C4.2, C5.2, C8.2, C9.2, U$1.VSS@1, U$1.VSS@2, U$1.VSS@3, U$1.VSS@4, U$1.VSS@5, U$1.VSSA
- new net VDD: C1.1, C10.1, C11.1, C12.1, C8.1, C9.1, U$1.VBAT, U$1.VDD@1, U$1.VDD@2, U$1.VDD@3, U$1.VDD@4, U$1.VDD@5
- new net VDDA: C2.1, C5.1, U$1.VDDA, U$1.VREF+
- net N$3: now also C3.1, U$1.VCAP2; no longer C1_V6.1, C2_V6.1, U$1.VDDA
- net N$4: now also C4.1, U$1.VCAP1; no longer C1_V3.1, C2_V3.1, U$1.VDD@3
Other:
- note added: "Ceramic Capacitor (Low ESR)"

Commit message: Bullshit
Parts:
- added C13, C14: (no value), resistor:C-USC0603
- added C15: 10uF, resistor:C-USC0603
- added C16, C_VBAT1: .1uF, resistor:C-USC0603
- added C17: 100nF, resistor:C-USC0603
- added C_VBAT2: 100uF, resistor:C-USC0603
- added L3, L4: 10uH, resistor:L-USL1812
- added U$2: TPS76850, TPSRegulators:TPS76850
- added U1: TPS73633DBVR, TPSRegulators:TPS73633DBVR
Connections:
- removed net VDD: C1.1, C10.1, C11.1, C12.1, C8.1, C9.1, U$1.VBAT, U$1.VDD@1, U$1.VDD@2, U$1.VDD@3, U$1.VDD@4, U$1.VDD@5
- removed net VDDA: C2.1, C5.1, U$1.VDDA, U$1.VREF+
- new net 3.3V: C1.1, C10.1, C11.1, C12.1, C15.1, C16.1, C8.1, C9.1, L4.1, U$1.VBAT, U$1.VDD@1, U$1.VDD@2, U$1.VDD@3, U$1.VDD@4, U$1.VDD@5, U1.OUT
- new net 5V: C13.1, C14.1, L3.2, U$2.OUT1, U$2.OUT2, U1.EN, U1.IN
- new net A3.3V: C2.1, C5.1, L4.2, U$1.VDDA, U$1.VREF+
- new net A5.0V: L3.1
- new net N$2: C17.1, U1.NR
- new net N$8: C13.2, C14.2, C16.2, U1.GND
- new net V_BAT: C_VBAT1.1, C_VBAT2.1, U$2.IN1, U$2.IN2
- net GND: now also C17.2, C_VBAT1.2, C_VBAT2.2, U$2.EN, U$2.GND
