File: eagle/master_schematic.sch (EAGLE design)
At the start: 22 parts, among them U1 TPS73633DBVR

Commit message: Merged into Master
Parts:
- added 1, U$6: MMBUTTON, MMButton:MMBUTTON
- added C6: 100uF, resistor:C-EUC1206
- added C7, C_L_L: 0.1uF, resistor:C-EUC1206
- added C_5V_3: 100uF, resistor:C-USC0603
- added C_L_R: 0.1 uF, resistor:C-EUC1206
- added LED1, LED2, LED3, LED4, LED5, LED6, LED7, LED8, LED9: SFH482, led:SFH482
- added LF_REC, L_REC, RF_REC, R_REC: BP103, opto-trans-siemens:BP103
- added PWR_LED: green, led:LED3MM
- added R1, R2: (no value), resistor:R-US_M1206
- added R10, R11, R3, R4, R5, R6, R7, R8, R9: 1k, resistor:R-US_R0805W
- added R_BT0_2, R_RST_UP: 47k, resistor:R-US_R1206
- added R_LF_R, R_L_R, R_RF_R, R_R_R: 1.8k ohm, resistor:R-US_R1206
- added R_PWR: 200 Ohm, resistor:R-US_M1206
- added U$3: TC44278MSOP, MMmosfet:TC44278MSOP
- added U$4: H-BRIDGE, MMHbridge:H-BRIDGE
- added U$5: 2X3HEADER, MM2x3Header:2X3HEADER
- C13: value (none) -> 0.1 uF; device resistor:C-USC0603 -> resistor:C-EUC0805K
- C_5V_4: value (none) -> .1uF
- renumbered C14 to C_5V_4
Connections:
- new net GND1: R1.1, R2.1, U$5.P$5
- new net LED1: R11.2
- new net LED2: R10.2
- new net LED3: R9.2
- new net LED4: R8.2
- new net LED5: R7.2
- new net LED6: R6.2
- new net LED7: R5.2
- new net LED8: R4.2
- new net LED9: R3.2
- new net N$1: PWR_LED.A, R_BT0_2.2, R_PWR.1, U$6.P$1
- new net N$10: U$4.P1S/P2S
- new net N$11: U$5.P$1
- new net N$12: U$3.OUT_A, U$4.N1G
- new net N$13: U$4.N2D/P2D, U$5.P$6
- new net N$14: U$3.OUT_B, U$4.N2G, U$4.P2G
- new net N$15: U$5.P$2
- new net N$16: U$5.P$3
- new net N$17: U$5.P$4
- new net N$18: LF_REC.E, R_LF_R.2
- new net N$19: L_REC.E, R_L_R.2
- new net N$20: R_REC.E, R_R_R.2
- new net N$21: RF_REC.E, R_RF_R.2
- new net N$22: LED1.A, R11.1
- new net N$23: LED2.A, R10.1
- new net N$24: LED3.A, R9.1
- new net N$25: LED4.A, R8.1
- new net N$26: C13.1, R_RST_UP.1
- new net N$27: 1.P$3
- new net N$28: LED5.A, R7.1
- new net N$29: U$6.P$2
- new net N$30: LED6.A, R6.1
- new net N$32: LED7.A, R5.1
- new net N$33: LED8.A, R4.1
- new net N$36: LED9.A, R3.1
- new net N$5: R1.2, U$3.IN_A
- new net N$6: R2.2, U$3.IN_B
- new net N$7: U$4.N1D/P1D
- new net N$9: U$4.P1G
- new net PE: 1.P$2, 1.P$4, C13.2, C6.1, C7.1, C_L_L.2, C_L_R.2, LED1.C, LED2.C, LED3.C, LED4.C, LED5.C, LED6.C, LED7.C, LED8.C, LED9.C, R_BT0_2.1, R_LF_R.1, R_L_R.1, R_RF_R.1, R_R_R.1, U$3.GND, U$4.N1S/N2S, U$6.P$3
- new net RESET: 1.P$1, R_RST_UP.2
- new net VA3.3: C_L_L.1, C_L_R.1, LF_REC.C, L_REC.C, RF_REC.C, R_REC.C
- net 3.3V: now also U$6.P$4
- net 5V: now also C_5V_3.1, R_PWR.2; no longer C13.1
- net GND: now also C15.2, C16.2, C_5V_3.2, C_5V_4.2, PWR_LED.C, U1.GND
- net N$8: now also C6.2, C7.2, U$3.VDD; no longer C13.2, C16.2, C_5V_4.2, U1.GND

Commit message: New Schematic
Parts:
- removed C13: 0.1 uF, resistor:C-EUC0805K
- added C14: 100uF, resistor:C-EUC1206
- added C18: 0.1uF, resistor:C-EUC1206
- added C_RESET: 0.1 uF, resistor:C-EUC0805K
- added R12, R13: (no value), resistor:R-US_M1206
- added U$7: TC44278MSOP, MMmosfet:TC44278MSOP
- added U$8: H-BRIDGE, MMHbridge:H-BRIDGE
- added U$9: 2X3HEADER, MM2x3Header:2X3HEADER
Connections:
- net N$11 renamed L_ENC_A
- net N$17 renamed L_ENC_B
- net N$5 renamed LPWMA
- net N$6 renamed LPWMB
- removed net N$10: U$4.P1S/P2S
- removed net N$15: U$5.P$2
- removed net N$26: C13.1, R_RST_UP.1
- removed net N$8: C6.2, C7.2, U$3.VDD
- removed net VA3.3: C_L_L.1, C_L_R.1, LF_REC.C, L_REC.C, RF_REC.C, R_REC.C
- new net BOOT0: R_BT0_2.2, U$6.P$1
- new net N$31: U$7.OUT_A, U$8.N1G
- new net N$34: U$7.OUT_B, U$8.N2G, U$8.P2G
- new net N$35: U$8.N1D/P1D
- new net N$37: U$8.P1G
- new net N$38: U$8.N2D/P2D, U$9.P$6
- new net N$39: U$9.P$3
- new net RPWMA: R12.2, U$7.IN_A
- new net RPWMB: R13.2, U$7.IN_B
- new net R_ENC_A: U$9.P$1
- new net R_ENC_B: U$9.P$4
- net 3.3V: now also R_RST_UP.2
- net 5V: now also U$5.P$2, U$9.P$2
- net A3.3V: now also C_L_L.1, C_L_R.1, LF_REC.C, L_REC.C, RF_REC.C, R_REC.C
- net GND: now also 1.P$2, 1.P$4, C_RESET.2, LED1.C, LED2.C, LED3.C, LED4.C, LED5.C, LED6.C, LED7.C, LED8.C, LED9.C, R_BT0_2.1, U$6.P$3
- net GND1: now also R12.1, R13.1, U$9.P$5
- net N$1: no longer R_BT0_2.2, U$6.P$1
- net PE: now also C14.1, C18.1, U$7.GND, U$8.N1S/N2S; no longer 1.P$2, 1.P$4, C13.2, LED1.C, LED2.C, LED3.C, LED4.C, LED5.C, LED6.C, LED7.C, LED8.C, LED9.C, R_BT0_2.1, U$6.P$3
- net RESET: now also C_RESET.1, R_RST_UP.1; no longer R_RST_UP.2
- net V_BAT: now also C14.2, C18.2, C6.2, C7.2, U$3.VDD, U$4.P1S/P2S, U$7.VDD, U$8.P1S/P2S
Other:
- moved on the sheet: R_RST_UP

Commit message: Schematic
Connections:
- net N$18 renamed LEFT_REC
- net N$19 renamed LF_REC
- net N$20 renamed RF_REC
- net N$21 renamed RIGHT_REC
- new net NRST: U$1.NRST
- new net SWCLK: U$1.PA14
- new net SWDIO: U$1.PA13
- new net TDS-SWO: U$1.PB3
- net BOOT0: now also U$1.BOOT0
- net LPWMA: now also U$1.PD12
- net LPWMB: now also U$1.PD13
- net RPWMA: now also U$1.PD14
- net RPWMB: now also U$1.PD15
Changed lines of the file:
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@@
 <label x="-454.66" y="-40.64" size="1.778" layer="95" rot="R180" xref="yes"/>
+</segment>
+<segment>
+<pinref part="U$1" gate="G$1" pin="PD14"/>
+<wire x1="83.82" y1="12.7" x2="88.9" y2="12.7" width="0.1524" layer="91"/>
+<label x="88.9" y="12.7" size="1.016" layer="95" xref="yes"/>
 </segment>
 </net>
@@
 <junction x="-429.26" y="-60.96"/>
 <label x="-454.66" y="-60.96" size="1.778" layer="95" rot="R180" xref="yes"/>
+</segment>
+<segment>
+<pinref part="U$1" gate="G$1" pin="PD15"/>
+<label x="93.98" y="15.24" size="1.016" layer="95" xref="yes"/>
+<wire x1="83.82" y1="15.24" x2="93.98" y2="15.24" width="0.1524" layer="91"/>
 </segment>
 </net>
@@
 </segment>
 </net>
-<net name="N$18" class="0">
+<net name="LEFT_REC" class="0">
 <segment>
 <pinref part="LF_REC" gate="1" pin="E"/>
@@
 </segment>
 </net>
-<net name="N$19" class="0">
+<net name="LF_REC" class="0">
 <segment>
 <pinref part="R_L_R" gate="G$1" pin="2"/>
@@
 </segment>
 </net>
-<net name="N$20" class="0">
+<net name="RF_REC" class="0">
 <segment>
 <pinref part="R_REC" gate="1" pin="E"/>
@@
 </segment>
 </net>
-<net name="N$21" class="0">
+<net name="RIGHT_REC" class="0">
 <segment>
 <pinref part="RF_REC" gate="1" pin="E"/>
@@
 <junction x="55.88" y="370.84"/>
 </segment>
+<segment>
+<pinref part="U$1" gate="G$1" pin="BOOT0"/>
+<wire x1="-71.12" y1="30.48" x2="-76.2" y2="30.48" width="0.1524" layer="91"/>
+<label x="-76.2" y="30.48" size="1.016" layer="95" rot="R180" xref="yes"/>
+</segment>
 </net>
 <net name="LPWMA" class="0">
@@
 <label x="-454.66" y="60.96" size="1.778" layer="95" rot="R180" xref="yes"/>
 </segment>
+<segment>
+<pinref part="U$1" gate="G$1" pin="PD12"/>
+<wire x1="83.82" y1="7.62" x2="88.9" y2="7.62" width="0.1524" layer="91"/>
+<label x="88.9" y="7.62" size="1.016" layer="95" xref="yes"/>
+</segment>
 </net>
 <net name="LPWMB" class="0">
@@
 <junction x="-429.26" y="40.64"/>
 <label x="-454.66" y="40.64" size="1.778" layer="95" rot="R180" xref="yes"/>
+</segment>
+<segment>
+<pinref part="U$1" gate="G$1" pin="PD13"/>
+<label x="93.98" y="10.16" size="1.016" layer="95" xref="yes"/>
+<wire x1="83.82" y1="10.16" x2="93.98" y2="10.16" width="0.1524" layer="91"/>
 </segment>
 </net>
@@
 </segment>
 </net>
+<net name="NRST" class="0">
+<segment>
+<pinref part="U$1" gate="G$1" pin="NRST"/>
+<wire x1="45.72" y1="12.7" x2="43.18" y2="12.7" width="0.1524" layer="91"/>
+<label x="43.18" y="12.7" size="1.016" layer="95" rot="R180" xref="yes"/>
+</segment>
+</net>
+<net name="SWDIO" class="0">
+<segment>
+<pinref part="U$1" gate="G$1" pin="PA13"/>
+<wire x1="83.82" y1="40.64" x2="88.9" y2="40.64" width="0.1524" layer="91"/>
+<label x="88.9" y="40.64" size="1.016" layer="95" xref="yes"/>
+</segment>
+</net>
+<net name="SWCLK" class="0">
+<segment>
+<pinref part="U$1" gate="G$1" pin="PA14"/>
+<wire x1="-71.12" y1="-15.24" x2="-76.2" y2="-15.24" width="0.1524" layer="91"/>
+<label x="-76.2" y="-15.24" size="1.016" layer="95" rot="R180" xref="yes"/>
+</segment>
+</net>
+<net name="TDS-SWO" class="0">
+<segment>
+<pinref part="U$1" gate="G$1" pin="PB3"/>
+<wire x1="-71.12" y1="17.78" x2="-76.2" y2="17.78" width="0.1524" layer="91"/>
+<label x="-76.2" y="17.78" size="1.016" layer="95" rot="R180" xref="yes"/>
+</segment>
+</net>

Commit message: New Schematic
Parts:
- removed 1, U$6: MMBUTTON, MMButton:MMBUTTON
- removed C_L_L: 0.1uF, resistor:C-EUC1206
- removed C_L_R: 0.1 uF, resistor:C-EUC1206
- removed C_RESET: 0.1 uF, resistor:C-EUC0805K
- removed LED5, LED6, LED7, LED8, LED9: SFH482, led:SFH482
- removed LF_REC, L_REC, RF_REC, R_REC: BP103, opto-trans-siemens:BP103
- removed R10, R11, R3, R4, R5, R6, R7, R8, R9: 1k, resistor:R-US_R0805W
- removed R_BT0_2, R_RST_UP: 47k, resistor:R-US_R1206
- removed R_LF_R, R_L_R, R_RF_R, R_R_R: 1.8k ohm, resistor:R-US_R1206
- removed U$4, U$8: H-BRIDGE, MMHbridge:H-BRIDGE
- removed U$5, U$9: 2X3HEADER, MM2x3Header:2X3HEADER
- removed U$7: TC44278MSOP, MMmosfet:TC44278MSOP
- added 2, U$16: MMBUTTON, MMButton:MMBUTTON
- added C13, C19, C20, C21, C22, C23: (no value), rcl:C-USC0603
- added C_L_L1: 0.1uF, resistor:C-EUC0603
- added C_L_R1, C_RESET1: 0.1 uF, resistor:C-EUC0603
- added LED10, LED11, LED12, LED13, LED14, LED15, LED16, LED17, LED18: SFH482, led:SFH482
- added LF_REC1, L_REC1, RF_REC1, R_REC1: BP103, opto-trans-siemens:BP103
- added R18, R19, R20, R21, R22, R23, R24, R25, R26: 1k, resistor:R-US_R0603
- added R_BT0_1, R_RST_UP1: 47k, resistor:R-US_R0603
- added R_LF_R1, R_L_R1, R_RF_R1, R_R_R1: 1.8k ohm, resistor:R-US_R0603
- added U$10, U$13: TC44278MSOP, MMmosfet:TC44278MSOP
- added U$11, U$14: H-BRIDGE, MMHbridge:H-BRIDGE
- added U$12, U$15: 2X3HEADER, MM2x3Header:2X3HEADER
- C1, C10, C11, C12, C2, C3, C4, C5, C8, C9: device rcl:C-USC1206 -> rcl:C-USC0603
- C14, C6: value 100uF -> 100nF; device resistor:C-EUC1206 -> rcl:C-EUC0603
- C18, C7: value 0.1uF -> 100nF; device resistor:C-EUC1206 -> rcl:C-EUC0603
- LED1, LED2, LED3, LED4: value SFH482 -> (none); device led:SFH482 -> led:LED5MM
- R1, R12, R13, R2: device resistor:R-US_M1206 -> resistor:R-US_R0603
- U$3: value TC44278MSOP -> ULN2003APWR; device MMmosfet:TC44278MSOP -> MMULN:ULN2003APWR
Connections:
- removed net N$12: U$3.OUT_A, U$4.N1G
- removed net N$13: U$4.N2D/P2D, U$5.P$6
- removed net N$14: U$3.OUT_B, U$4.N2G, U$4.P2G
- removed net N$16: U$5.P$3
- removed net N$22: LED1.A, R11.1
- removed net N$23: LED2.A, R10.1
- removed net N$24: LED3.A, R9.1
- removed net N$25: LED4.A, R8.1
- removed net N$27: 1.P$3
- removed net N$28: LED5.A, R7.1
- removed net N$29: U$6.P$2
- removed net N$30: LED6.A, R6.1
- removed net N$31: U$7.OUT_A, U$8.N1G
- removed net N$32: LED7.A, R5.1
- removed net N$33: LED8.A, R4.1
- removed net N$34: U$7.OUT_B, U$8.N2G, U$8.P2G
- removed net N$35: U$8.N1D/P1D
- removed net N$36: LED9.A, R3.1
- removed net N$37: U$8.P1G
- removed net N$38: U$8.N2D/P2D, U$9.P$6
- removed net N$39: U$9.P$3
- removed net N$7: U$4.N1D/P1D
- removed net N$9: U$4.P1G
- new net N$10: U$11.P1G
- new net N$11: U$11.N2D/P2D, U$12.P$6
- new net N$15: U$12.P$3
- new net N$17: U$13.OUT_A, U$14.N1G
- new net N$18: U$13.OUT_B, U$14.N2G, U$14.P2G
- new net N$19: U$14.N1D/P1D
- new net N$20: U$14.P1G
- new net N$21: U$14.N2D/P2D, U$15.P$6
- new net N$26: U$15.P$3
- new net N$40: LED18.A, R26.1
- new net N$41: LED17.A, R25.1
- new net N$42: LED16.A, R24.1
- new net N$43: LED15.A, R23.1
- new net N$44: LED14.A, R22.1
- new net N$45: LED13.A, R21.1
- new net N$46: LED12.A, R20.1
- new net N$47: LED11.A, R19.1
- new net N$48: LED10.A, R18.1
- new net N$49: 2.P$3
- new net N$5: U$10.OUT_A, U$11.N1G
- new net N$50: U$16.P$2
- new net N$6: U$10.OUT_B, U$11.N2G, U$11.P2G
- new net N$8: U$11.N1D/P1D
- net 3.3V: now also R_RST_UP1.2, U$16.P$4; no longer R_RST_UP.2, U$6.P$4
- net 5V: now also U$12.P$2, U$15.P$2; no longer U$5.P$2, U$9.P$2
- net A3.3V: now also C_L_L1.1, C_L_R1.1, LF_REC1.C, L_REC1.C, RF_REC1.C, R_REC1.C; no longer C_L_L.1, C_L_R.1, LF_REC.C, L_REC.C, RF_REC.C, R_REC.C
- net BOOT0: now also R_BT0_1.2, U$16.P$1; no longer R_BT0_2.2, U$6.P$1
- net GND: now also 2.P$2, 2.P$4, C_RESET1.2, LED10.C, LED11.C, LED12.C, LED13.C, LED14.C, LED15.C, LED16.C, LED17.C, LED18.C, R_BT0_1.1, U$16.P$3; no longer 1.P$2, 1.P$4, C_RESET.2, LED1.C, LED2.C, LED3.C, LED4.C, LED5.C, LED6.C, LED7.C, LED8.C, LED9.C, R_BT0_2.1, U$6.P$3
- net GND1: now also U$12.P$5, U$15.P$5; no longer U$5.P$5, U$9.P$5
- net LED1: now also R26.2; no longer R11.2
- net LED2: now also R25.2; no longer R10.2
- net LED3: now also R24.2; no longer R9.2
- net LED4: now also R23.2; no longer R8.2
- net LED5: now also R22.2; no longer R7.2
- net LED6: now also R21.2; no longer R6.2
- net LED7: now also R20.2; no longer R5.2
- net LED8: now also R19.2; no longer R4.2
- net LED9: now also R18.2; no longer R3.2
- net LEFT_REC: now also LF_REC1.E, R_LF_R1.2; no longer LF_REC.E, R_LF_R.2
- net LF_REC: now also L_REC1.E, R_L_R1.2; no longer L_REC.E, R_L_R.2
- net LPWMA: now also R12.2, U$10.IN_A; no longer R1.2, U$3.IN_A
- net LPWMB: now also R13.2, U$10.IN_B; no longer R2.2, U$3.IN_B
- net L_ENC_A: now also U$12.P$1; no longer U$5.P$1
- net L_ENC_B: now also U$12.P$4; no longer U$5.P$4
- net PE: now also C_L_L1.2, C_L_R1.2, R_LF_R1.1, R_L_R1.1, R_RF_R1.1, R_R_R1.1, U$10.GND, U$11.N1S/N2S, U$13.GND, U$14.N1S/N2S; no longer C_L_L.2, C_L_R.2, R_LF_R.1, R_L_R.1, R_RF_R.1, R_R_R.1, U$3.GND, U$4.N1S/N2S, U$7.GND, U$8.N1S/N2S
- net RESET: now also 2.P$1, C_RESET1.1, R_RST_UP1.1; no longer 1.P$1, C_RESET.1, R_RST_UP.1
- net RF_REC: now also R_REC1.E, R_R_R1.2; no longer R_REC.E, R_R_R.2
- net RIGHT_REC: now also RF_REC1.E, R_RF_R1.2; no longer RF_REC.E, R_RF_R.2
- net RPWMA: now also R1.2, U$13.IN_A; no longer R12.2, U$7.IN_A
- net RPWMB: now also R2.2, U$13.IN_B; no longer R13.2, U$7.IN_B
- net R_ENC_A: now also U$15.P$1; no longer U$9.P$1
- net R_ENC_B: now also U$15.P$4; no longer U$9.P$4
- net V_BAT: now also U$10.VDD, U$11.P1S/P2S, U$13.VDD, U$14.P1S/P2S; no longer U$3.VDD, U$4.P1S/P2S, U$7.VDD, U$8.P1S/P2S

Commit message: Organization
Connections:
- new net LED1-: U$1.PE9
- new net LF_TX: U$1.PE6
- new net L_TX: U$1.PE5
- new net N$12: U$1.PE7
- new net N$13: U$1.PB2
- new net N$14: U$1.PA1
- new net N$16: U$1.PA2
- new net N$9: U$1.PE8
- new net RF_TX: U$1.PD8
- new net RX: U$1.PA10
- new net R_TX: U$1.PD9
- new net TX: U$1.PA9
- net GND: no longer 2.P$2, U$16.P$3
- net LED1: now also U$1.PD6
- net LED2: now also U$1.PE11
- net LED3: now also U$1.PE12
- net LED7: now also U$1.PB14
- net LED8: now also U$1.PB13
- net LED9: now also U$1.PB12
- net LEFT_REC: now also U$1.PA6
- net LF_REC: now also U$1.PC5
- net LPWMA: now also U$1.PA3
- net L_ENC_A: now also U$1.PE2
- net L_ENC_B: now also U$1.PE3
- net RF_REC: now also U$1.PC4
- net RIGHT_REC: now also U$1.PA7
- net RPWMA: now also U$1.PA0-WKUP
- net R_ENC_A: now also U$1.PC8
- net R_ENC_B: now also U$1.PC9
Other:
- note added: "Pin 22 and 25 are TIM2 Pins"
- note added: "Pins 30-33 are ADC Pins"
- note added: "Pins 59 - 62 are TIM4 pins"
- moved on the sheet: C1, C10, C11, C12, C14, C15, C16, C17, C18, C2, C3, C4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

Commit message: stuff
Parts:
- removed 2, U$16: MMBUTTON, MMButton:MMBUTTON
- removed LED1, LED2, LED3, LED4: (no value), led:LED5MM
- removed U$12, U$15: 2X3HEADER, MM2x3Header:2X3HEADER
- removed U$3: ULN2003APWR, MMULN:ULN2003APWR
- added BOOT0, RST, S2, S3: (no value), switch-omron:10-XX
- added C_RESET2, C_RESET3: 0.1 uF, resistor:C-EUC0603
- added JP1, JP2: (no value), pinhead:PINHD-2X3
- added JP3, JP4: (no value), pinhead:PINHD-1X2
- added R3, R6: 10 ohm, resistor:R-US_R1206
- added R4, R5: 6 ohm, resistor:R-US_R1206
- added R_SW1, R_SW2: 47k, resistor:R-US_R0603
- added U$4: ULN2003APWR, MMULN:ULN2003APWR
- C13, C19, C20, C21, C22, C23: device rcl:C-USC0603 -> resistor:C-EUC1206
Connections:
- removed net N$26: U$15.P$3
- removed net N$49: 2.P$3
- removed net N$50: U$16.P$2
- new net LF_EMITTER: U$4.7B
- new net L_EMITTER: U$4.5B, U$4.6B
- new net N$22: R3.1, U$4.2C
- new net N$23: R3.2
- new net N$24: R4.1, U$4.3C, U$4.4C
- new net N$25: R4.2
- new net N$27: R5.1, U$4.5C, U$4.6C
- new net N$28: R5.2
- new net N$29: R6.2
- new net N$30: R6.1, U$4.7C
- new net N$31: JP3.1
- new net N$7: U$4.1C
- new net RF_EMITTER: U$4.2B
- new net R_EMITTER: U$4.3B, U$4.4B
- net 3.3V: now also BOOT0.P, S2.P, S3.P; no longer U$16.P$4
- net 5V: now also C13.1, C19.1, C20.1, C21.1, C22.1, C23.1, JP1.3, JP2.3; no longer U$12.P$2, U$15.P$2
- net BOOT0: now also BOOT0.S; no longer U$16.P$1
- net GND: now also JP4.2, RST.P, R_SW1.1, R_SW2.1; no longer 2.P$4
- net GND1: now also JP1.4, JP2.4; no longer U$12.P$5, U$15.P$5
- net L_ENC_A: now also JP2.1; no longer U$12.P$1
- net L_ENC_B: now also JP2.2; no longer U$12.P$4
- net N$11: now also JP2.6; no longer U$12.P$6
- net N$15: now also JP3.2, JP4.1; no longer U$12.P$3
- net N$19: now also JP1.5
- net N$21: now also JP1.6; no longer U$15.P$6
- net N$8: now also JP2.5
- net PE: now also C13.2, C19.2, C20.2, C21.2, C22.2, C23.2, U$4.E
- net RESET: now also RST.S; no longer 2.P$1
- net R_ENC_A: now also JP1.1; no longer U$15.P$1
- net R_ENC_B: now also JP1.2; no longer U$15.P$4
Other:
- note added: "ULN2003APWR"
- moved on the sheet: C13, C19, C20, C21, C22, C23
