File: eagle/master_schematic.sch (EAGLE design)
At the start: 90 parts, among them U1 TPS73633DBVR

Commit message: Switch
Parts:
- added SW1: (no value), special:SW_DIP-1
Connections:
- new net N$26: C_RESET2.2, R_SW1.2, S3.S
- new net N$32: C_RESET3.2, R_SW2.2, S2.S
- new net N$33: C_RESET2.1
- new net N$34: C_RESET3.1
- net V_BAT: now also SW1.1
Other:
- moved on the sheet: C_RESET2, C_RESET3, C_VBAT2, S2, S3
Changed lines of the file:
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@@
 <?xml version="1.0" encoding="utf-8"?>
 <!DOCTYPE eagle SYSTEM "eagle.dtd">
-<eagle version="7.6.0">
+<eagle version="7.2.0">
 <drawing>
 <settings>
@@
 <part name="R_SW1" library="resistor" deviceset="R-US_" device="R0603" value="47k"/>
 <part name="R_SW2" library="resistor" deviceset="R-US_" device="R0603" value="47k"/>
+<part name="SW1" library="special" deviceset="SW_DIP-1" device=""/>
 </parts>
 <sheets>
@@
 <instance part="U$2" gate="G$1" x="-83.82" y="35.56"/>
 <instance part="SUPPLY1" gate="GND" x="-114.3" y="45.72"/>
-<instance part="C_VBAT2" gate="G$1" x="-109.22" y="2.54"/>
+<instance part="C_VBAT2" gate="G$1" x="-121.92" y="2.54"/>
 <instance part="C_VBAT1" gate="G$1" x="-96.52" y="2.54"/>
 <instance part="C_5V_3" gate="G$1" x="-17.78" y="2.54"/>
@@
 <instance part="L4" gate="G$1" x="104.14" y="25.4" rot="R90"/>
 <instance part="SUPPLY7" gate="GND" x="55.88" y="-20.32"/>
-<instance part="SUPPLY8" gate="GND" x="-109.22" y="-15.24"/>
+<instance part="SUPPLY8" gate="GND" x="-121.92" y="-15.24"/>
 <instance part="R_PWR" gate="G$1" x="-38.1" y="15.24" rot="R90"/>
 <instance part="PWR_LED" gate="G$1" x="-38.1" y="2.54"/>
 <instance part="JP3" gate="G$1" x="-162.56" y="17.78"/>
 <instance part="JP4" gate="G$1" x="-162.56" y="2.54"/>
+<instance part="SW1" gate="G$1" x="-152.4" y="40.64"/>
 </instances>
 <busses>
@@
 <segment>
 <pinref part="U$2" gate="G$1" pin="IN1"/>
-<wire x1="-101.6" y1="33.02" x2="-116.84" y2="33.02" width="0.1524" layer="91"/>
-<wire x1="-116.84" y1="33.02" x2="-116.84" y2="38.1" width="0.1524" layer="91"/>
+<wire x1="-101.6" y1="33.02" x2="-121.92" y2="33.02" width="0.1524" layer="91"/>
+<wire x1="-121.92" y1="33.02" x2="-121.92" y2="40.64" width="0.1524" layer="91"/>
 <pinref part="U$2" gate="G$1" pin="IN2"/>
-<wire x1="-101.6" y1="25.4" x2="-116.84" y2="25.4" width="0.1524" layer="91"/>
-<wire x1="-116.84" y1="25.4" x2="-116.84" y2="33.02" width="0.1524" layer="91"/>
-<junction x="-116.84" y="33.02"/>
-<label x="-116.84" y="38.1" size="1.778" layer="95" rot="R180" xref="yes"/>
+<wire x1="-101.6" y1="25.4" x2="-121.92" y2="25.4" width="0.1524" layer="91"/>
+<wire x1="-121.92" y1="25.4" x2="-121.92" y2="33.02" width="0.1524" layer="91"/>
+<junction x="-121.92" y="33.02"/>
+<label x="-121.92" y="40.64" size="1.778" layer="95" rot="R90" xref="yes"/>
 <pinref part="C_VBAT2" gate="G$1" pin="1"/>
-<wire x1="-109.22" y1="5.08" x2="-116.84" y2="5.08" width="0.1524" layer="91"/>
-<wire x1="-116.84" y1="5.08" x2="-116.84" y2="15.24" width="0.1524" layer="91"/>
-<junction x="-116.84" y="25.4"/>
+<wire x1="-121.92" y1="5.08" x2="-121.92" y2="15.24" width="0.1524" layer="91"/>
+<junction x="-121.92" y="25.4"/>
 <pinref part="C_VBAT1" gate="G$1" pin="1"/>
-<wire x1="-116.84" y1="15.24" x2="-116.84" y2="25.4" width="0.1524" layer="91"/>
+<wire x1="-121.92" y1="15.24" x2="-121.92" y2="25.4" width="0.1524" layer="91"/>
 <wire x1="-96.52" y1="5.08" x2="-96.52" y2="15.24" width="0.1524" layer="91"/>
-<wire x1="-96.52" y1="15.24" x2="-116.84" y2="15.24" width="0.1524" layer="91"/>
-<junction x="-116.84" y="15.24"/>
+<wire x1="-96.52" y1="15.24" x2="-121.92" y2="15.24" width="0.1524" layer="91"/>
+<junction x="-121.92" y="15.24"/>
+<pinref part="SW1" gate="G$1" pin="1"/>
+<wire x1="-144.78" y1="40.64" x2="-121.92" y2="40.64" width="0.1524" layer="91"/>
+<junction x="-121.92" y="40.64"/>
 </segment>
 </net>
@@
 <pinref part="C_VBAT2" gate="G$1" pin="2"/>
 <pinref part="SUPPLY8" gate="GND" pin="GND"/>
-<wire x1="-109.22" y1="-2.54" x2="-109.22" y2="-7.62" width="0.1524" layer="91"/>
+<wire x1="-121.92" y1="-2.54" x2="-121.92" y2="-7.62" width="0.1524" layer="91"/>
 <pinref part="C_VBAT1" gate="G$1" pin="2"/>
-<wire x1="-109.22" y1="-7.62" x2="-109.22" y2="-12.7" width="0.1524" layer="91"/>
+<wire x1="-121.92" y1="-7.62" x2="-121.92" y2="-12.7" width="0.1524" layer="91"/>
 <wire x1="-96.52" y1="-2.54" x2="-96.52" y2="-7.62" width="0.1524" layer="91"/>
-<wire x1="-96.52" y1="-7.62" x2="-109.22" y2="-7.62" width="0.1524" layer="91"/>
-<junction x="-109.22" y="-7.62"/>
+<wire x1="-96.52" y1="-7.62" x2="-121.92" y2="-7.62" width="0.1524" layer="91"/>
+<junction x="-121.92" y="-7.62"/>
 <pinref part="JP4" gate="G$1" pin="2"/>
 <wire x1="-165.1" y1="2.54" x2="-175.26" y2="2.54" width="0.1524" layer="91"/>
 <wire x1="-175.26" y1="2.54" x2="-175.26" y2="-7.62" width="0.1524" layer="91"/>
-<wire x1="-175.26" y1="-7.62" x2="-109.22" y2="-7.62" width="0.1524" layer="91"/>
+<wire x1="-175.26" y1="-7.62" x2="-121.92" y2="-7.62" width="0.1524" layer="91"/>
 </segment>
 <segment>
@@
 <pinref part="JP3" gate="G$1" pin="1"/>
 <wire x1="-165.1" y1="20.32" x2="-175.26" y2="20.32" width="0.1524" layer="91"/>
-<wire x1="-175.26" y1="20.32" x2="-175.26" y2="33.02" width="0.1524" layer="91"/>
-<wire x1="-175.26" y1="33.02" x2="-137.16" y2="33.02" width="0.1524" layer="91"/>
-<wire x1="-137.16" y1="33.02" x2="-137.16" y2="20.32" width="0.1524" layer="91"/>
+<wire x1="-175.26" y1="20.32" x2="-175.26" y2="40.64" width="0.1524" layer="91"/>
+<wire x1="-175.26" y1="40.64" x2="-160.02" y2="40.64" width="0.1524" layer="91"/>
 </segment>
 </net>
@@
 <instance part="SUPPLY27" gate="GND" x="-66.04" y="-58.42"/>
 <instance part="BOOT0" gate="1" x="76.2" y="10.16" rot="R270"/>
-<instance part="S2" gate="1" x="172.72" y="10.16" rot="R270"/>
-<instance part="S3" gate="1" x="129.54" y="10.16" rot="R270"/>
+<instance part="S2" gate="1" x="154.94" y="10.16" rot="R270"/>
+<instance part="S3" gate="1" x="119.38" y="10.16" rot="R270"/>
 <instance part="RST" gate="1" x="25.4" y="10.16" rot="R270"/>
-<instance part="C_RESET2" gate="G$1" x="116.84" y="30.48"/>
-<instance part="C_RESET3" gate="G$1" x="149.86" y="30.48"/>
+<instance part="C_RESET2" gate="G$1" x="127" y="25.4"/>
+<instance part="C_RESET3" gate="G$1" x="162.56" y="25.4"/>
 <instance part="R_SW1" gate="G$1" x="104.14" y="-12.7" rot="R90"/>
 <instance part="R_SW2" gate="G$1" x="134.62" y="-12.7" rot="R90"/>
@@
 <segment>
 <pinref part="S3" gate="1" pin="P"/>
-<wire x1="124.46" y1="10.16" x2="121.92" y2="10.16" width="0.1524" layer="91"/>
-<label x="121.92" y="10.16" size="1.778" layer="95" rot="R180" xref="yes"/>
+<wire x1="114.3" y1="10.16" x2="111.76" y2="10.16" width="0.1524" layer="91"/>
+<label x="109.22" y="10.16" size="1.778" layer="95" rot="R180" xref="yes"/>
+<wire x1="111.76" y1="10.16" x2="109.22" y2="10.16" width="0.1524" layer="91"/>
+<wire x1="116.84" y1="10.16" x2="111.76" y2="10.16" width="0.1524" layer="91"/>
+<wire x1="111.76" y1="10.16" x2="109.22" y2="10.16" width="0.1524" layer="91"/>
+<wire x1="111.76" y1="10.16" x2="109.22" y2="10.16" width="0.1524" layer="91"/>
 </segment>
 <segment>
 <pinref part="S2" gate="1" pin="P"/>
-<wire x1="167.64" y1="10.16" x2="165.1" y2="10.16" width="0.1524" layer="91"/>
-<label x="165.1" y="10.16" size="1.778" layer="95" rot="R180" xref="yes"/>
+<wire x1="149.86" y1="10.16" x2="144.78" y2="10.16" width="0.1524" layer="91"/>
+<label x="144.78" y="10.16" size="1.778" layer="95" rot="R180" xref="yes"/>
 </segment>
 </net>
@@
 </segment>
 </net>
+<net name="N$26" class="0">
+<segment>
+<pinref part="S3" gate="1" pin="S"/>
+<wire x1="124.46" y1="10.16" x2="127" y2="10.16" width="0.1524" layer="91"/>
+<wire x1="127" y1="10.16" x2="127" y2="-7.62" width="0.1524" layer="91"/>
+<pinref part="R_SW1" gate="G$1" pin="2"/>
+<wire x1="127" y1="-7.62" x2="104.14" y2="-7.62" width="0.1524" layer="91"/>
+<junction x="127" y="10.16"/>
+<pinref part="C_RESET2" gate="G$1" pin="2"/>
+<wire x1="127" y1="20.32" x2="127" y2="10.16" width="0.1524" layer="91"/>
+</segment>
+</net>
+<net name="N$32" class="0">
+<segment>
+<pinref part="R_SW2" gate="G$1" pin="2"/>
+<wire x1="134.62" y1="-7.62" x2="162.56" y2="-7.62" width="0.1524" layer="91"/>
+<wire x1="162.56" y1="-7.62" x2="162.56" y2="10.16" width="0.1524" layer="91"/>
+<pinref part="S2" gate="1" pin="S"/>
+<wire x1="162.56" y1="10.16" x2="160.02" y2="10.16" width="0.1524" layer="91"/>
+<junction x="162.56" y="10.16"/>
+<pinref part="C_RESET3" gate="G$1" pin="2"/>
+<wire x1="162.56" y1="20.32" x2="162.56" y2="10.16" width="0.1524" layer="91"/>
+</segment>
+</net>
+<net name="N$33" class="0">
+<segment>
+<pinref part="C_RESET2" gate="G$1" pin="1"/>
+<wire x1="127" y1="27.94" x2="127" y2="58.42" width="0.1524" layer="91"/>
+<label x="127" y="58.42" size="1.778" layer="95" font="vector" rot="R90" xref="yes"/>
+</segment>
+</net>
+<net name="N$34" class="0">
+<segment>
+<pinref part="C_RESET3" gate="G$1" pin="1"/>
+<wire x1="162.56" y1="27.94" x2="162.56" y2="58.42" width="0.1524" layer="91"/>
+<label x="162.56" y="58.42" size="1.778" layer="95" font="vector" rot="R90" xref="yes"/>
+</segment>
+</net>

Commit message: Comments
Parts:
- added JP5: (no value), pinhead:PINHD-2X3
Connections:
- removed net LED1-: U$1.PE9
- removed net N$26: C_RESET2.2, R_SW1.2, S3.S
- removed net N$32: C_RESET3.2, R_SW2.2, S2.S
- removed net N$33: C_RESET2.1
- removed net N$34: C_RESET3.1
- removed net N$9: U$1.PE8
- removed net NRST: U$1.NRST
- new net US_1: C_RESET2.1, R_SW1.1, S3.S, U$1.PE9
- new net US_2: C_RESET3.1, R_SW2.1, S2.S, U$1.PE8
- new net VDD: JP5.1
- net 3.3V: now also R_SW1.2, R_SW2.2; no longer S2.P, S3.P
- net GND: now also C_RESET2.2, C_RESET3.2, JP5.2, S2.P, S3.P; no longer R_SW1.1, R_SW2.1
- net LED4: now also U$1.PD1
- net LED5: now also U$1.PD2
- net LED6: now also U$1.PD3
- net RESET: now also U$1.NRST
- net RX: now also JP5.4
- net SWCLK: now also JP5.6
- net SWDIO: now also JP5.5
- net TX: now also JP5.3
Other:
- note added: "3.3V Low Dropout Regulator"
- note added: "5V Low-Dropout Regulator"
- note added: "Battery1"
- note added: "Battery2"
- note added: "Current Amplifier"
- note added: "Decoupling Capacitors (One at Every Vdd/Vss Pair)"
- note added: "Flash Mode Switch (Low - User Program High - Bootloader)"
- note added: "On/Off Switch"
- note added: "Power Indicator"
- note added: "Programming Headers"
- note added: "Reset Switch"
- note added: "User Switch 1 (Normally High)"
- note added: "User Switch 2 (Normally High)"
- moved on the sheet: C_RESET2, C_RESET3, R_SW1, R_SW2, S2
