File: eagle/master_schematic.sch (EAGLE design)
At the start: 110 parts

Commit message: Schematic Update
Parts:
- removed LED6, LED7, LED8, LED9: (no value), led:LEDCHIPLED_0603
- removed R_LED6, R_LED7, R_LED8, R_LED9: 1k, resistor:R-US_R0603
- removed R_LEFT, R_RIGHT: 6 ohm, resistor:R-US_R1206
- removed R_LF, R_RF: 10 ohm, resistor:R-US_R1206
- added R_LF_E, R_RF_E: 10 ohm, resistor:R-US_R0603
- added R_L_E, R_R_E: 6 ohm, resistor:R-US_R0603
- C1_F_EMITS, C1_L_EMIT, C1_R_EMIT, C2_F_EMITS, C2_L_EMIT, C2_R_EMIT: device resistor:C-EUC1206 -> resistor:C-EUC0603
- LED1, LED2, LED3, LED4, LED5: device led:LEDCHIPLED_0603 -> led:LEDCHIPLED_0805
- R1_VOLT, R2_VOLT: device resistor:R-US_R0805 -> resistor:R-US_R0603
- R_PWR: device resistor:R-US_M0805 -> resistor:R-US_R0603
- renumbered C_VCAP3 to C_VCAP1, C_VCAP4 to C_VCAP2, D1 to D_G, D2 to D_B, L2 to L33, L3 to L50, R_LF_R1 to R_L_R, R_L_R1 to R_LF_R, R_RF_R1 to R_R_R, R_R_R1 to R_RF_R, S3 to S1
Connections:
- removed net GND1: C1_LMOT.1, C1_RMOT.1, C2_LMOT.1, C2_RMOT.1, HB_L.N1S/N2S, HB_R.N1S/N2S, L_MOT.4, MOS_L.GND, MOS_R.GND, R1_LMOT.1, R1_RMOT.1, R2_LMOT.1, R2_RMOT.1, R_MOT.4
- removed net LED6: R_LED6.2, U$3.PD4
- removed net LED7: R_LED7.2, U$3.PD3
- removed net LED8: R_LED8.2, U$3.PD2
- removed net LED9: R_LED9.2, U$3.PD1
- removed net N$22: R_RF.1, U$9.2C
- removed net N$30: R_LF.1, U$9.7C
- removed net N$45: LED6.A, R_LED6.1
- removed net N$46: LED7.A, R_LED7.1
- removed net N$47: LED8.A, R_LED8.1
- removed net N$48: LED9.A, R_LED9.1
- new net N$13: R_R_E.1, U$9.7C
- new net N$4: R_L_E.1, U$9.2C
- net GND: now also C1_LMOT.1, C1_RMOT.1, C2_LMOT.1, C2_RMOT.1, HB_L.N1S/N2S, HB_R.N1S/N2S, L_MOT.4, MOS_L.GND, MOS_R.GND, R1_LMOT.1, R1_RMOT.1, R2_LMOT.1, R2_RMOT.1, R_MOT.4; no longer LED6.C, LED7.C, LED8.C, LED9.C
- net LF_EMITTER: now also U$3.PC9; no longer U$3.PB4
- net L_EMITTER: now also U$3.PC8; no longer U$3.PB5
- net N$23: now also R_RF_E.2; no longer R_RF.2
- net N$24: now also R_LF_E.1; no longer R_RIGHT.1
- net N$25: now also R_R_E.2; no longer R_RIGHT.2
- net N$26: now also R_L_E.2; no longer R_LEFT.2
- net N$27: now also R_RF_E.1; no longer R_LEFT.1
- net N$28: now also R_LF_E.2; no longer R_LF.2
- net RF_EMITTER: now also U$3.PB5; no longer U$3.PC9
- net R_EMITTER: now also U$3.PB4; no longer U$3.PC8
