File: eagle/rev2/rev2.sch (EAGLE design)
At the start: 102 parts

Commit message: hex file
Parts:
- removed U$1: BAT, mounts:BAT
- C1_LMOT, C1_RMOT, C2_LMOT, C2_RMOT: device rcl:C-EUC0603 -> rcl:C-EUC0805
- C_VBAT2: device resistor:C-USC0603 -> resistor:C-USC1206
Connections:
- net 3.3V: now also PROG_HEAD.2; no longer PROG_HEAD.6
- net GND: now also PROG_HEAD.4; no longer PROG_HEAD.8
- net LED1: now also U$3.PD1; no longer U$3.PB12
- net LED2: now also U$3.PD2; no longer U$3.PB13
- net LED3: now also U$3.PD3; no longer U$3.PB14
- net LED4: now also U$3.PD4; no longer U$3.PC2
- net LED5: now also U$3.PD5; no longer U$3.PC1
- net LPWMA: now also U$3.PA0-WKUP; no longer U$3.PA2
- net LPWMB: now also U$3.PA1; no longer U$3.PA3
- net RPWMA: now also U$3.PA2; no longer U$3.PA0-WKUP
- net RPWMB: now also U$3.PA3; no longer U$3.PA1
- net SWCLK: now also PROG_HEAD.6; no longer PROG_HEAD.4
- net SWDIO: now also PROG_HEAD.8; no longer PROG_HEAD.2

Commit message: Clean directory
Parts:
- removed R1_VOLT: 20k, resistor:R-US_R0603
- removed R2_VOLT: 10k, resistor:R-US_R0603
- removed U$5: MOTOR, mounts:MOTOR
- U$3: value STM32F769VG-1 -> STM32F746VG
Connections:
- removed net VOLTMETER: R1_VOLT.1, R2_VOLT.2, U$3.PC0
- net GND: no longer R2_VOLT.1
- net LENCA: now also U$3.PE9; no longer U$3.PE11
- net LENCB: now also U$3.PE11; no longer U$3.PE9
- net RENCA: now also U$3.PE13; no longer U$3.PE14
- net RENCB: now also U$3.PE14; no longer U$3.PE13
- net V_BAT: no longer R1_VOLT.2
Other:
- moved on the sheet: C1_A, C1_BAT, C2_A, C_1, C_2, C_3, C_4, C_5, PROG_HEAD
