File: MouseRev100000/MoueRev3.brd (EAGLE design)
At the start: 103.7 x 74.8 mm, 93 parts

Commit message: Final Board
Parts:
- added LED8: (no value), led:CHIPLED_0805
- added R_LED8: 1k, resistor:R0603
Connections:
- removed net N$17: HB_R.N1G, MOS_R.OUT_A
- new net LED9: R_LED8.2, U$3.52
- new net N$12: LED8.C
- new net N$16: LED8.A, R_LED8.1
- new net N$7: HB_R.N1G, HB_R.P1G, MOS_R.OUT_A
Routing:
- net N$7: track 0.00 -> 22.7 mm, vias 0 -> 2
- net N$17: track 6.12 -> 0.00 mm
- net LED9: track 0.00 -> 2.89 mm
- net N$16: track 0.00 -> 2.24 mm
- net A5.0V: track 79.2 -> 81.1 mm
- net V_BAT: track 126.8 -> 128.0 mm
Other:
- outline, holes or cut-outs redrawn
- board text added: "Should have used an Arduino"

Commit message: Apparently this is the final PCB
Parts:
- added LED6, LED7, LED9: (no value), led:CHIPLED_0805
- added R_LED6, R_LED7, R_LED9: 1k, resistor:R0603
- moved C_1 33.4 mm to (87.9, 60.5), turned to 180 degrees
- moved C_3 20.7 mm to (68.0, 57.7)
- moved C_2 17.3 mm to (87.9, 39.3), turned to 270 degrees
- moved C2_A 17.0 mm to (82.0, 40.0), turned to 180 degrees
- moved R_LED4 15.3 mm to (39.9, 40.0)
- moved LED4 15.1 mm to (36.1, 40.1)
- moved R_LED3 14.3 mm to (39.9, 38.0)
- moved LED3 13.8 mm to (36.1, 38.1)
- moved R_LED2 13.8 mm to (39.9, 35.3)
- moved C1_A 13.5 mm to (82.0, 38.1), turned to 180 degrees
- moved R_LED1 13.4 mm to (39.9, 32.5)
- moved LED2 13.1 mm to (36.3, 35.3)
- moved C_RREC 13.1 mm to (26.1, 82.6)
- moved LED1 12.8 mm to (36.3, 32.5)
- moved R_REC 12.1 mm to (22.4, 79.0)
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Connections:
- removed net N$12: LED8.C
- new net GND: C_RESET1.2, LED1.C, LED2.C, LED3.C, LED4.C, LED5.C, LED6.C, LED7.C, LED8.C, LED9.C, RST.3, R_BT0_1.1
- new net LED10: R_LED9.2, U$3.80
- new net LED11: R_LED7.2, U$3.79
- new net LED12: R_LED6.2, U$3.78
- new net N$17: LED6.A, R_LED6.1
- new net N$30: LED7.A, R_LED7.1
- new net N$33: LED9.A, R_LED9.1
- net N$3: no longer C_RESET1.2, LED1.C, LED2.C, LED3.C, LED4.C, LED5.C, RST.3, R_BT0_1.1
Routing:
- net GND: track 0.00 -> 114.3 mm, vias 0 -> 4
- net LED12: track 0.00 -> 32.5 mm
- net LED11: track 0.00 -> 32.1 mm
- net LED10: track 0.00 -> 30.7 mm
- net 5V: track 231.9 -> 256.2 mm, vias 2 -> 1
- net LED3: track 24.3 -> 39.8 mm
- net LED2: track 26.2 -> 41.6 mm
- net LED1: track 29.2 -> 43.9 mm
- net LED4: track 23.8 -> 38.3 mm
- net 3.3V: track 216.7 -> 202.3 mm, vias 2 -> 3
- net N$3: track 187.4 -> 173.3 mm, vias 18 -> 15
- net RIGHT_REC: track 82.0 -> 95.4 mm
- net N$57: track 23.5 -> 10.0 mm
- net N$25: track 35.0 -> 26.4 mm
- net LEFT_REC: track 83.2 -> 90.5 mm
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Other:
- board text added: "Rome wasn't built in a day but it was burnt down in one."
- board text added: "The Frat Rat"
