File: MouseRev100000/MoueRev3.sch (EAGLE design)
At the start: 92 parts

Commit message: Final Board
Parts:
- added LED8: (no value), led:LEDCHIPLED_0805
- added R_LED8: 1k, resistor:R-US_R0603
Connections:
- removed net N$17: HB_R.N1G, MOS_R.OUT_A
- new net LED9: R_LED8.2, U$3.PB13
- new net N$12: LED8.C
- new net N$16: LED8.A, R_LED8.1
- new net N$7: HB_R.N1G, HB_R.P1G, MOS_R.OUT_A
Changed lines of the file:
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@@
 <part name="U$8" library="JST_CONNECTOR_FEMALE. through hole" deviceset="JST_CONNECTOR_FEMALE" device=""/>
 <part name="U$9" library="ULN2003APWR" deviceset="ULN2003APWR" device=""/>
+<part name="R_LED8" library="resistor" deviceset="R-US_" device="R0603" value="1k"/>
+<part name="LED8" library="led" deviceset="LED" device="CHIPLED_0805"/>
 </parts>
 <sheets>
@@
 <wire x1="-15.24" y1="0" x2="-15.24" y2="7.62" width="0.1524" layer="91"/>
 <label x="-15.24" y="7.62" size="1.27" layer="95" rot="R90" xref="yes"/>
+</segment>
+</net>
+<net name="LED9" class="0">
+<segment>
+<pinref part="U$3" gate="G$1" pin="PB13"/>
+<wire x1="40.64" y1="-73.66" x2="50.8" y2="-73.66" width="0.1524" layer="91"/>
+<label x="50.8" y="-73.66" size="1.27" layer="95" xref="yes"/>
 </segment>
 </net>
@@
 </segment>
 </net>
-<net name="N$17" class="0">
-<segment>
-<pinref part="MOS_R" gate="G$1" pin="OUT_A"/>
-<junction x="-33.02" y="-43.18"/>
-<wire x1="-33.02" y1="-43.18" x2="-17.78" y2="-43.18" width="0.1524" layer="91"/>
-<wire x1="-17.78" y1="-43.18" x2="-17.78" y2="-15.24" width="0.1524" layer="91"/>
-<wire x1="-17.78" y1="-15.24" x2="-5.08" y2="-15.24" width="0.1524" layer="91"/>
-<pinref part="HB_R" gate="G$1" pin="N1G"/>
-</segment>
-</net>
 <net name="N$18" class="0">
 <segment>
@@
 <pinref part="L_MOT" gate="A" pin="3"/>
 <wire x1="50.8" y1="66.04" x2="68.58" y2="66.04" width="0.1524" layer="91"/>
+</segment>
+</net>
+<net name="N$7" class="0">
+<segment>
+<pinref part="HB_R" gate="G$1" pin="P1G"/>
+<junction x="30.48" y="-15.24"/>
+<wire x1="30.48" y1="-15.24" x2="33.02" y2="-15.24" width="0.1524" layer="91"/>
+<wire x1="33.02" y1="-15.24" x2="33.02" y2="7.62" width="0.1524" layer="91"/>
+<pinref part="MOS_R" gate="G$1" pin="OUT_A"/>
+<junction x="-33.02" y="-43.18"/>
+<wire x1="-33.02" y1="-43.18" x2="-17.78" y2="-43.18" width="0.1524" layer="91"/>
+<wire x1="-17.78" y1="-43.18" x2="-17.78" y2="-15.24" width="0.1524" layer="91"/>
+<wire x1="-17.78" y1="-15.24" x2="-7.62" y2="-15.24" width="0.1524" layer="91"/>
+<pinref part="HB_R" gate="G$1" pin="N1G"/>
+<wire x1="-7.62" y1="-15.24" x2="-5.08" y2="-15.24" width="0.1524" layer="91"/>
+<wire x1="33.02" y1="7.62" x2="-7.62" y2="7.62" width="0.1524" layer="91"/>
+<wire x1="-7.62" y1="7.62" x2="-7.62" y2="-15.24" width="0.1524" layer="91"/>
+<junction x="-7.62" y="-15.24"/>
 </segment>
 </net>
@@
 <instance part="LED4" gate="G$1" x="-55.88" y="-25.4"/>
 <instance part="LED5" gate="G$1" x="-66.04" y="-25.4"/>
+<instance part="R_LED8" gate="G$1" x="-96.52" y="-7.62" rot="R90"/>
+<instance part="LED8" gate="G$1" x="-96.52" y="-25.4"/>
 </instances>
 <busses>
@@
 <junction x="-55.88" y="-30.48"/>
 <junction x="-66.04" y="-30.48"/>
+<wire x1="-78.74" y1="-38.1" x2="-66.04" y2="-38.1" width="0.1524" layer="91"/>
+<wire x1="50.8" y1="-38.1" x2="101.6" y2="-38.1" width="0.1524" layer="91"/>
+<junction x="50.8" y="-38.1"/>
 </segment>
 </net>
@@
 <pinref part="R_LED4" gate="G$1" pin="2"/>
 <junction x="-55.88" y="-2.54"/>
-<label x="-55.88" y="15.24" size="1.778" layer="95" rot="R90" xref="yes"/>
 <wire x1="-55.88" y1="15.24" x2="-55.88" y2="-2.54" width="0.1524" layer="91"/>
+<label x="-55.88" y="15.24" size="1.27" layer="95" rot="R90" xref="yes"/>
 </segment>
 </net>
@@
 <pinref part="R_LED5" gate="G$1" pin="2"/>
 <junction x="-66.04" y="-2.54"/>
-<label x="-66.04" y="15.24" size="1.778" layer="95" rot="R90" xref="yes"/>
 <wire x1="-66.04" y1="15.24" x2="-66.04" y2="-2.54" width="0.1524" layer="91"/>
+<label x="-66.04" y="15.24" size="1.27" layer="95" rot="R90" xref="yes"/>
 </segment>
 </net>
@@
 </segment>
 </net>
+<net name="N$12" class="0">
+<segment>
+<wire x1="-96.52" y1="-38.1" x2="-96.52" y2="-30.48" width="0.1524" layer="91"/>
+<wire x1="-73.66" y1="-38.1" x2="-96.52" y2="-38.1" width="0.1524" layer="91"/>
+<pinref part="LED8" gate="G$1" pin="C"/>
+<junction x="-96.52" y="-30.48"/>
+</segment>
+</net>
+<net name="N$16" class="0">
+<segment>
+<pinref part="R_LED8" gate="G$1" pin="1"/>
+<junction x="-96.52" y="-12.7"/>
+<wire x1="-96.52" y1="-12.7" x2="-96.52" y2="-22.86" width="0.1524" layer="91"/>
+<pinref part="LED8" gate="G$1" pin="A"/>
+<junction x="-96.52" y="-22.86"/>
+</segment>
+</net>
+<net name="LED9" class="0">
+<segment>
+<pinref part="R_LED8" gate="G$1" pin="2"/>
+<junction x="-96.52" y="-2.54"/>
+<label x="-96.52" y="15.24" size="1.778" layer="95" rot="R90" xref="yes"/>
+<wire x1="-96.52" y1="15.24" x2="-96.52" y2="-2.54" width="0.1524" layer="91"/>
+</segment>
+</net>

Commit message: Apparently this is the final PCB
Parts:
- added LED6, LED7, LED9: (no value), led:LEDCHIPLED_0805
- added R_LED6, R_LED7, R_LED9: 1k, resistor:R-US_R0603
Connections:
- removed net N$12: LED8.C
- new net GND: C_RESET1.2, LED1.C, LED2.C, LED3.C, LED4.C, LED5.C, LED6.C, LED7.C, LED8.C, LED9.C, RST.P, R_BT0_1.1
- new net LED10: R_LED9.2, U$3.PC12
- new net LED11: R_LED7.2, U$3.PC11
- new net LED12: R_LED6.2, U$3.PC10
- new net N$17: LED6.A, R_LED6.1
- new net N$30: LED7.A, R_LED7.1
- new net N$33: LED9.A, R_LED9.1
- net N$3: no longer C_RESET1.2, LED1.C, LED2.C, LED3.C, LED4.C, LED5.C, RST.P, R_BT0_1.1
Other:
- moved on the sheet: LED8, R_LED8
